File: schematic/espRFID.sch (KiCad schematic (older format))
At the start: 17 parts

Commit message: Merge Dev (#3)
* Add KiCAD files to .gitignore

* Ignore DS_Store on Mac OS

* Move code to separate directory

* Remove redundant PIO ignores

Platform.io auto-generates own ignore file, base directory had redundant 
ignore.

* Fix SecretConstants header and include base c++ file

* Change pio.ini to include arduino library dirs on Mac OS

* Add template c++ file for SecretConstants

* Add extra KiCAD files to .gitignore

* Update libary references for KiCAD 5.0+

* Cleanup schematic in prep for additional work

* Add required libraries to PlatformIO config

* Update install instructions in README.md
Parts:
- C? (x2): symbol CP1 -> Device:CP1
- D?: symbol LED -> espRFID-rescue:LED
- D? (x2): symbol D -> Device:D
- JP?: symbol JUMPER3 -> espRFID-rescue:JUMPER3
- P?: symbol CONN_01X03 -> espRFID-rescue:CONN_01X03
- P? (x4): symbol CONN_01X02 -> espRFID-rescue:CONN_01X02
- Q? (x2): symbol Q_NMOS_GDS -> Device:Q_NMOS_GDS
- R?: symbol R -> Device:R
- U?: symbol RDM6300 -> rdm6300:RDM6300
- U?: symbol WiMos_D1_mini -> wimos_d1_mini:WiMos_D1_mini
- U?: symbol 7805 -> espRFID-rescue:7805
Connections:
- wire segments 53 -> 61
